File: kicad/modules/control_panel_module/indicators.kicad_sch (KiCad schematic)
At the start: 0 parts

Commit message: add control panel module
Parts:
- added D1: LED_GREEN, LED_SMD:LED_0603_1608Metric_Pad1.05x0.95mm_HandSolder, symbol Device:LED
- added D2: LED_ORANGE, LED_SMD:LED_0603_1608Metric_Pad1.05x0.95mm_HandSolder, symbol Device:LED
- added D3: LED_RED, LED_SMD:LED_0603_1608Metric_Pad1.05x0.95mm_HandSolder, symbol Device:LED
- added LED_ERR_OFFBOARD1, LED_STATUS_OFFBOARD1: Screw_Terminal_01x02, TerminalBlock_MetzConnect:TerminalBlock_MetzConnect_Type101_RT01602HBWC_1x02_P5.08mm_Horizontal, symbol Connector:Screw_Terminal_01x02
- added R4, R5, R6: 1k, Resistor_SMD:R_0603_1608Metric_Pad0.98x0.95mm_HandSolder, symbol Device:R
- added U1: ULN2004A, Package_SO:SOIC-16W_5.3x10.2mm_P1.27mm, symbol Transistor_Array:ULN2004A
Connections:
- new net: LED_ERR_OFFBOARD1.2 (Pin_2), U1.10 (O7), U1.11 (O6), U1.12 (O5)
- new net: D1.2 (A), R4.2
- new net: D2.2 (A), R5.2
- new net: D3.2 (A), R6.2
- new net: LED_STATUS_OFFBOARD1.2 (Pin_2), U1.13 (O4), U1.14 (O3), U1.15 (O2), U1.16 (O1)
- new net +3.3V: R4.1
- new net +Vin: LED_ERR_OFFBOARD1.1 (Pin_1), LED_STATUS_OFFBOARD1.1 (Pin_1), U1.9 (COM)
- new net ERR: R6.1, U1.5 (I5), U1.6 (I6), U1.7 (I7)
- new net GND: D1.1 (K), D2.1 (K), D3.1 (K), U1.8 (GND)
- new net STATUS: R5.1, U1.1 (I1), U1.2 (I2), U1.3 (I3), U1.4 (I4)
