File: kicad/modules/control_panel_module/SSD1306.kicad_sch (KiCad schematic)
At the start: 1 part

Commit message: Add part numbers
Parts:
- Brd1: Manufacturer Part Number (none) -> 333099; Mouser number (none) -> 392-333099
Changed lines of the file:
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@@
 			)
 		)
-		(property "Description" "SSD1306 OLED"
+		(property "Description" "CUSTOM"
 			(at 101.6 72.39 0)
 			(effects
@@
 			)
 		)
-		(property "Manufacturer Part Number" ""
+		(property "Manufacturer Part Number" "333099"
 			(at 101.6 72.39 0)
 			(effects
@@
 			)
 		)
-		(property "Mouser number" ""
+		(property "Mouser number" "392-333099"
 			(at 101.6 72.39 0)
 			(effects
