File: kicad/modules/control_panel_module/buttons.kicad_sch (KiCad schematic)
At the start: 5 parts

Commit message: Connector for bigger current, control module 2
Parts:
- RV_SPEED2: Mouser number (none) -> 688-RK09D1130F30B104
- SW_MODE1: Mouser number (none) -> 653-B3FS1095P
Changed lines of the file:
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@@
+			)
+		)
+		(property "Manufacturer Part Number" ""
+			(at 153.67 64.77 0)
+			(effects
+				(font
+					(size 1.27 1.27)
+				)
+				(hide yes)
+			)
+		)
+		(property "Mouser number" ""
+			(at 153.67 64.77 0)
+			(effects
+				(font
+					(size 1.27 1.27)
+				)
+				(hide yes)
 			)
 		)
@@
 			)
 		)
-		(property "Description" "688-RK09D1130F30B104"
+		(property "Description" ""
+			(at 59.69 67.31 0)
+			(effects
+				(font
+					(size 1.27 1.27)
+				)
+				(hide yes)
+			)
+		)
+		(property "Manufacturer Part Number" ""
+			(at 59.69 67.31 0)
+			(effects
+				(font
+					(size 1.27 1.27)
+				)
+				(hide yes)
+			)
+		)
+		(property "Mouser number" "688-RK09D1130F30B104"
 			(at 59.69 67.31 0)
 			(effects
@@
 			)
 		)
+		(property "Manufacturer Part Number" ""
+			(at 43.18 67.31 0)
+			(effects
+				(font
+					(size 1.27 1.27)
+				)
+				(hide yes)
+			)
+		)
+		(property "Mouser number" ""
+			(at 43.18 67.31 0)
+			(effects
+				(font
+					(size 1.27 1.27)
+				)
+				(hide yes)
+			)
+		)
 		(pin "1"
 		)
@@
 			)
 		)
+		(property "Manufacturer Part Number" ""
+			(at 83.82 67.31 0)
+			(effects
+				(font
+					(size 1.27 1.27)
+				)
+				(hide yes)
+			)
+		)
+		(property "Mouser number" ""
+			(at 83.82 67.31 0)
+			(effects
+				(font
+					(size 1.27 1.27)
+				)
+				(hide yes)
+			)
+		)
 		(pin "2"
 		)
@@
 			)
 		)
-		(property "Description" "653-B3FS1095P"
+		(property "Description" ""
 			(at 125.73 68.58 0)
 			(effects
+				(font
+					(size 1.27 1.27)
+				)
+				(hide yes)
+			)
+		)
+		(property "Manufacturer Part Number" ""
+			(at 125.73 68.58 0)
+			(effects
+				(font
+					(size 1.27 1.27)
+				)
+				(hide yes)
+			)
+		)
+		(property "Mouser number" "653-B3FS1095P"
+			(at 125.73 68.58 0)
+			(effects

Commit message: Add part numbers
Parts:
- J5: renamed from RV_SPEED1; value Screw_Terminal_01x03 -> 1x3 5.08; Manufacturer Part Number (none) -> TB0012-508-03GR; Mouser number (none) -> 179-TB0012-508-03GR
- J6: renamed from SW_MODE2; value Screw_Terminal_01x02 -> 1x2 5.08; Manufacturer Part Number (none) -> TB0012-508-02GR; Mouser number (none) -> 179-TB0012-508-02GR
- JP1: value Jumper_3_Bridged12 -> 1x3 2.54; Manufacturer Part Number (none) -> 68000-420HLF; Mouser number (none) -> 649-68000-420HLF
- RV1: renamed from RV_SPEED2; Manufacturer Part Number (none) -> RK09D1130-F30-C0-B104
- SW1: renamed from SW_MODE1; Manufacturer Part Number (none) -> B3FS-1095P
Changed lines of the file:
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@@
 		(dnp no)
 		(fields_autoplaced yes)
-		(property "Reference" "SW_MODE2"
+		(property "Reference" "J6"
 			(at 156.21 64.7699 0)
 			(effects
@@
 			)
 		)
-		(property "Value" "Screw_Terminal_01x02"
+		(property "Value" "1x2 5.08"
 			(at 156.21 67.3099 0)
 			(effects
@@
 			)
 		)
-		(property "Description" "Generic screw terminal, single row, 01x02, script generated (kicad-library-utils/schlib/autogen/connector/)"
+		(property "Description" "CUSTOM"
 			(at 153.67 64.77 0)
 			(effects
@@
 			)
 		)
-		(property "Manufacturer Part Number" ""
+		(property "Manufacturer Part Number" "TB0012-508-02GR"
 			(at 153.67 64.77 0)
 			(effects
@@
 			)
 		)
-		(property "Mouser number" ""
+		(property "Mouser number" "179-TB0012-508-02GR"
 			(at 153.67 64.77 0)
 			(effects
@@
 			(project "control_panel_module"
 				(path "/01f48663-51d7-48f4-9aa9-9279c565a6cb/f1f09a98-6452-4cc9-9ea6-171d66ed561a"
-					(reference "SW_MODE2")
+					(reference "J6")
 					(unit 1)
 				)
@@
 		(on_board yes)
 		(dnp no)
-		(property "Reference" "RV_SPEED2"
+		(property "Reference" "RV1"
 			(at 71.374 59.69 0)
 			(effects
@@
 			)
 		)
-		(property "Description" ""
+		(property "Description" "CUSTOM"
 			(at 59.69 67.31 0)
 			(effects
@@
 			)
 		)
-		(property "Manufacturer Part Number" ""
+		(property "Manufacturer Part Number" "RK09D1130-F30-C0-B104 "
 			(at 59.69 67.31 0)
 			(effects
@@
 			(project "control_panel_module"
 				(path "/01f48663-51d7-48f4-9aa9-9279c565a6cb/f1f09a98-6452-4cc9-9ea6-171d66ed561a"
-					(reference "RV_SPEED2")
+					(reference "RV1")
 					(unit 1)
 				)
@@
 		(on_board yes)
 		(dnp no)
-		(property "Reference" "RV_SPEED1"
+		(property "Reference" "J5"
 			(at 42.926 76.2 0)
 			(effects
@@
 			)
 		)
-		(property "Value" "Screw_Terminal_01x03"
+		(property "Value" "1x3 5.08"
 			(at 36.83 73.914 0)
 			(effects
@@
 			)
 		)
-		(property "Description" "Generic screw terminal, single row, 01x03, script generated (kicad-library-utils/schlib/autogen/connector/)"
+		(property "Description" "CUSTOM"
 			(at 43.18 67.31 0)
 			(effects
@@
 			)
 		)
-		(property "Manufacturer Part Number" ""
+		(property "Manufacturer Part Number" "TB0012-508-03GR"
 			(at 43.18 67.31 0)
 			(effects
@@
 			)
 		)
-		(property "Mouser number" ""
+		(property "Mouser number" " 179-TB0012-508-03GR"
 			(at 43.18 67.31 0)
 			(effects
@@
 			(project "control_panel_module"
 				(path "/01f48663-51d7-48f4-9aa9-9279c565a6cb/f1f09a98-6452-4cc9-9ea6-171d66ed561a"
-					(reference "RV_SPEED1")
+					(reference "J5")
 					(unit 1)
 				)
@@
 			)
 		)
-		(property "Value" "Jumper_3_Bridged12"
+		(property "Value" "1x3 2.54"
 			(at 83.82 71.628 0)
 			(effects
@@
 			)
 		)
-		(property "Description" "Jumper, 3-pole, pins 1+2 closed/bridged"
+		(property "Description" "CUSTOM"
 			(at 83.82 67.31 0)
 			(effects
@@
 			)
 		)
-		(property "Manufacturer Part Number" ""
+		(property "Manufacturer Part Number" "68000-420HLF"
 			(at 83.82 67.31 0)
 			(effects
@@
 			)
 		)
-		(property "Mouser number" ""
+		(property "Mouser number" "649-68000-420HLF"
 			(at 83.82 67.31 0)
 			(effects
@@
 		(on_board yes)
 		(dnp no)
-		(property "Reference" "SW_MODE1"
+		(property "Reference" "SW1"
 			(at 125.476 65.278 0)
 			(effects
@@
 			)
 		)
-		(property "Description" ""
+		(property "Description" "CUSTOM"
 			(at 125.73 68.58 0)
 			(effects
@@
 			)
 		)
-		(property "Manufacturer Part Number" ""
+		(property "Manufacturer Part Number" "B3FS-1095P "
 			(at 125.73 68.58 0)
 			(effects
@@
 			(project "control_panel_module"
 				(path "/01f48663-51d7-48f4-9aa9-9279c565a6cb/f1f09a98-6452-4cc9-9ea6-171d66ed561a"
-					(reference "SW_MODE1")
-					(unit 1)
-				)
+					(reference "SW1")
+					(unit 1)
+				)

Commit message: BOM with Ullmanna part numbers
Changed lines of the file:
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@@
 (kicad_sch
-	(version 20231120)
+	(version 20250114)
 	(generator "eeschema")
-	(generator_version "8.0")
+	(generator_version "9.0")
 	(paper "A5")
 	(junction
@@
 		(shape output)
 		(at 83.82 60.96 90)
-		(fields_autoplaced yes)
 		(effects
 			(font
@@
 		(shape output)
 		(at 115.57 68.58 180)
-		(fields_autoplaced yes)
 		(effects
 			(font
@@
 			)
 		)
+		(property "Ullmanna Part Number" ""
+			(at 153.67 64.77 0)
+			(effects
+				(font
+					(size 1.27 1.27)
+				)
+				(hide yes)
+			)
+		)
 		(pin "1"
 		)
@@
 		)
 		(property "Mouser number" "688-RK09D1130F30B104"
+			(at 59.69 67.31 0)
+			(effects
+				(font
+					(size 1.27 1.27)
+				)
+				(hide yes)
+			)
+		)
+		(property "Ullmanna Part Number" ""
 			(at 59.69 67.31 0)
 			(effects
@@
 			)
 		)
+		(property "Ullmanna Part Number" ""
+			(at 43.18 67.31 0)
+			(effects
+				(font
+					(size 1.27 1.27)
+				)
+				(hide yes)
+			)
+		)
 		(pin "1"
 		)
@@
 			)
 		)
+		(property "Ullmanna Part Number" ""
+			(at 83.82 67.31 0)
+			(effects
+				(font
+					(size 1.27 1.27)
+				)
+				(hide yes)
+			)
+		)
 		(pin "2"
 		)
@@
 			(at 125.73 68.58 0)
 			(effects
+				(font
+					(size 1.27 1.27)
+				)
+				(hide yes)
+			)
+		)
+		(property "Ullmanna Part Number" ""
+			(at 125.73 68.58 0)
+			(effects
