File: kicad/modules/control_panel_module/control_panel_module.kicad_sch (KiCad schematic)
At the start: 2 parts, among them J1 Screw_Terminal_01x06, J2 Screw_Terminal_01x06

Commit message: Add part numbers
Parts:
- J1, J2: value Screw_Terminal_01x06 -> 1x6 2.54; Manufacturer Part Number (none) -> 68000-420HLF; Mouser number (none) -> 649-68000-420HLF
Changed lines of the file:
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@@
 			)
 		)
-		(property "Value" "Screw_Terminal_01x06"
+		(property "Value" "1x6 2.54"
 			(at 68.58 91.44 0)
 			(effects
@@
 			)
 		)
-		(property "Description" "Generic screw terminal, single row, 01x06, script generated (kicad-library-utils/schlib/autogen/connector/)"
-			(at 68.58 80.01 0)
-			(effects
-				(font
-					(size 1.27 1.27)
-				)
-				(hide yes)
-			)
-		)
-		(property "Manufacturer Part Number" ""
-			(at 68.58 80.01 0)
-			(effects
-				(font
-					(size 1.27 1.27)
-				)
-				(hide yes)
-			)
-		)
-		(property "Mouser number" ""
+		(property "Description" "CUSTOM"
+			(at 68.58 80.01 0)
+			(effects
+				(font
+					(size 1.27 1.27)
+				)
+				(hide yes)
+			)
+		)
+		(property "Manufacturer Part Number" "68000-420HLF"
+			(at 68.58 80.01 0)
+			(effects
+				(font
+					(size 1.27 1.27)
+				)
+				(hide yes)
+			)
+		)
+		(property "Mouser number" "649-68000-420HLF"
 			(at 68.58 80.01 0)
 			(effects
@@
 			)
 		)
-		(property "Value" "Screw_Terminal_01x06"
+		(property "Value" "1x6 2.54"
 			(at 68.58 49.53 0)
 			(effects
@@
 			)
 		)
-		(property "Description" "Generic screw terminal, single row, 01x06, script generated (kicad-library-utils/schlib/autogen/connector/)"
-			(at 68.58 38.1 0)
-			(effects
-				(font
-					(size 1.27 1.27)
-				)
-				(hide yes)
-			)
-		)
-		(property "Manufacturer Part Number" ""
-			(at 68.58 38.1 0)
-			(effects
-				(font
-					(size 1.27 1.27)
-				)
-				(hide yes)
-			)
-		)
-		(property "Mouser number" ""
-			(at 68.58 38.1 0)
-			(effects
+		(property "Description" "CUSTOM"
+			(at 68.58 38.1 0)
+			(effects
+				(font
+					(size 1.27 1.27)
+				)
+				(hide yes)
+			)
+		)
+		(property "Manufacturer Part Number" "68000-420HLF"
+			(at 68.58 38.1 0)
+			(effects
+				(font
+					(size 1.27 1.27)
+				)
+				(hide yes)
+			)
+		)
+		(property "Mouser number" "649-68000-420HLF"
+			(at 68.58 38.1 0)
+			(effects
