File: kicad/Impact_driver_controller/current_probe.kicad_sch (KiCad schematic)
At the start: 5 parts, among them U2 ACS712 30A

Commit message: Connector for bigger current, control module 2
Parts:
- C2: Mouser Part Number (none) -> 80-C0603C102J2TAUTO
- R1, R2, R3: Mouser Part Number (none) -> 71-CRCW0603-10K-E3
- U2: Mouser Part Number (none) -> 250-712ELCTR30AT
Changed lines of the file:
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@@
 			)
 		)
-		(property "Description" "71-CRCW0603-10K-E3"
+		(property "Description" ""
+			(at 123.19 78.74 0)
+			(effects
+				(font
+					(size 1.27 1.27)
+				)
+				(hide yes)
+			)
+		)
+		(property "Manufacturer Part Number" ""
+			(at 123.19 78.74 0)
+			(effects
+				(font
+					(size 1.27 1.27)
+				)
+				(hide yes)
+			)
+		)
+		(property "Mouser Part Number" "71-CRCW0603-10K-E3"
 			(at 123.19 78.74 0)
 			(effects
@@
 			)
 		)
-		(property "Description" "71-CRCW0603-10K-E3"
+		(property "Description" ""
+			(at 123.19 59.69 0)
+			(effects
+				(font
+					(size 1.27 1.27)
+				)
+				(hide yes)
+			)
+		)
+		(property "Manufacturer Part Number" ""
+			(at 123.19 59.69 0)
+			(effects
+				(font
+					(size 1.27 1.27)
+				)
+				(hide yes)
+			)
+		)
+		(property "Mouser Part Number" "71-CRCW0603-10K-E3"
 			(at 123.19 59.69 0)
 			(effects
@@
 			)
 		)
-		(property "Description" "80-C0603C102J2TAUTO"
+		(property "Description" ""
+			(at 105.41 60.96 0)
+			(effects
+				(font
+					(size 1.27 1.27)
+				)
+				(hide yes)
+			)
+		)
+		(property "Manufacturer Part Number" ""
+			(at 105.41 60.96 0)
+			(effects
+				(font
+					(size 1.27 1.27)
+				)
+				(hide yes)
+			)
+		)
+		(property "Mouser Part Number" "80-C0603C102J2TAUTO"
 			(at 105.41 60.96 0)
 			(effects
@@
 			)
 		)
-		(property "Description" "71-CRCW0603-10K-E3"
+		(property "Description" ""
+			(at 123.19 69.85 0)
+			(effects
+				(font
+					(size 1.27 1.27)
+				)
+				(hide yes)
+			)
+		)
+		(property "Manufacturer Part Number" ""
+			(at 123.19 69.85 0)
+			(effects
+				(font
+					(size 1.27 1.27)
+				)
+				(hide yes)
+			)
+		)
+		(property "Mouser Part Number" "71-CRCW0603-10K-E3"
 			(at 123.19 69.85 0)
 			(effects
@@
 			)
 		)
-		(property "Description" "250-712ELCTR30AT"
+		(property "Description" ""
 			(at 86.36 52.07 0)
 			(effects
+				(font
+					(size 1.27 1.27)
+				)
+				(hide yes)
+			)
+		)
+		(property "Manufacturer Part Number" ""
+			(at 86.36 52.07 0)
+			(effects
+				(font
+					(size 1.27 1.27)
+				)
+				(hide yes)
+			)
+		)
+		(property "Mouser Part Number" "250-712ELCTR30AT"
+			(at 86.36 52.07 0)
+			(effects

Commit message: Add part numbers
Parts:
- C2: Manufacturer Part Number (none) -> C0603C102J2TACAUTO
- R1, R2, R3: Manufacturer Part Number (none) -> CRCW060310K0FKEA
- U2: value ACS712 30A -> ACS71230A; Manufacturer Part Number (none) -> ACS712ELCTR-30A-T
Changed lines of the file:
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@@
 			)
 		)
-		(property "Description" ""
+		(property "Description" "ULM"
 			(at 123.19 78.74 0)
 			(effects
@@
 			)
 		)
-		(property "Manufacturer Part Number" ""
+		(property "Manufacturer Part Number" "CRCW060310K0FKEA"
 			(at 123.19 78.74 0)
 			(effects
@@
 			)
 		)
-		(property "Description" ""
+		(property "Description" "ULM"
 			(at 123.19 59.69 0)
 			(effects
@@
 			)
 		)
-		(property "Manufacturer Part Number" ""
+		(property "Manufacturer Part Number" "CRCW060310K0FKEA"
 			(at 123.19 59.69 0)
 			(effects
@@
 			)
 		)
-		(property "Description" ""
+		(property "Description" "CUSTOM"
 			(at 105.41 60.96 0)
 			(effects
@@
 			)
 		)
-		(property "Manufacturer Part Number" ""
+		(property "Manufacturer Part Number" "C0603C102J2TACAUTO"
 			(at 105.41 60.96 0)
 			(effects
@@
 			)
 		)
-		(property "Description" ""
+		(property "Description" "ULM"
 			(at 123.19 69.85 0)
 			(effects
@@
 			)
 		)
-		(property "Manufacturer Part Number" ""
+		(property "Manufacturer Part Number" "CRCW060310K0FKEA"
 			(at 123.19 69.85 0)
 			(effects
@@
 			)
 		)
-		(property "Value" "ACS712 30A"
+		(property "Value" "ACS71230A"
 			(at 88.5541 41.91 0)
 			(effects
@@
 			)
 		)
-		(property "Description" ""
+		(property "Description" "CUSTOM"
 			(at 86.36 52.07 0)
 			(effects
@@
 			)
 		)
-		(property "Manufacturer Part Number" ""
+		(property "Manufacturer Part Number" "ACS712ELCTR-30A-T"
 			(at 86.36 52.07 0)
 			(effects

Commit message: BOM with Ullmanna part numbers
Parts:
- C2: Manufacturer Part Number C0603C102J2TACAUTO -> GRM1885C1H102JA01D; Mouser Part Number 80-C0603C102J2TAUTO -> 81-GRM39C102J50; Ullmanna Part Number (none) -> BMCCK300
- R1, R2, R3: Manufacturer Part Number CRCW060310K0FKEA -> RC0603FR-0710KL; Mouser Part Number 71-CRCW0603-10K-E3 -> 603-RC0603FR-0710KL; Ullmanna Part Number (none) -> BMCR0201
Changed lines of the file:
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@@
 (kicad_sch
-	(version 20231120)
+	(version 20250114)
 	(generator "eeschema")
-	(generator_version "8.0")
+	(generator_version "9.0")
 	(paper "A5")
 	(junction
@@
 		(shape input)
 		(at 72.39 46.99 180)
-		(fields_autoplaced yes)
 		(effects
 			(font
@@
 		(shape output)
 		(at 72.39 57.15 180)
-		(fields_autoplaced yes)
 		(effects
 			(font
@@
 		(shape output)
 		(at 132.08 64.77 0)
-		(fields_autoplaced yes)
 		(effects
 			(font
@@
 			)
 		)
-		(property "Manufacturer Part Number" "CRCW060310K0FKEA"
+		(property "Manufacturer Part Number" "RC0603FR-0710KL"
 			(at 123.19 78.74 0)
 			(effects
@@
 			)
 		)
-		(property "Mouser Part Number" "71-CRCW0603-10K-E3"
+		(property "Mouser Part Number" "603-RC0603FR-0710KL"
+			(at 123.19 78.74 0)
+			(effects
+				(font
+					(size 1.27 1.27)
+				)
+				(hide yes)
+			)
+		)
+		(property "Ullmanna Part Number" "BMCR0201"
 			(at 123.19 78.74 0)
 			(effects
@@
 			)
 		)
-		(property "Manufacturer Part Number" "CRCW060310K0FKEA"
+		(property "Manufacturer Part Number" "RC0603FR-0710KL"
 			(at 123.19 59.69 0)
 			(effects
@@
 			)
 		)
-		(property "Mouser Part Number" "71-CRCW0603-10K-E3"
+		(property "Mouser Part Number" "603-RC0603FR-0710KL"
+			(at 123.19 59.69 0)
+			(effects
+				(font
+					(size 1.27 1.27)
+				)
+				(hide yes)
+			)
+		)
+		(property "Ullmanna Part Number" "BMCR0201"
 			(at 123.19 59.69 0)
 			(effects
@@
 			)
 		)
-		(property "Description" "CUSTOM"
+		(property "Description" "ULM"
 			(at 105.41 60.96 0)
 			(effects
@@
 			)
 		)
-		(property "Manufacturer Part Number" "C0603C102J2TACAUTO"
+		(property "Manufacturer Part Number" "GRM1885C1H102JA01D"
 			(at 105.41 60.96 0)
 			(effects
@@
 			)
 		)
-		(property "Mouser Part Number" "80-C0603C102J2TAUTO"
+		(property "Mouser Part Number" "81-GRM39C102J50"
+			(at 105.41 60.96 0)
+			(effects
+				(font
+					(size 1.27 1.27)
+				)
+				(hide yes)
+			)
+		)
+		(property "Ullmanna Part Number" "BMCCK300"
 			(at 105.41 60.96 0)
 			(effects
@@
 			)
 		)
-		(property "Manufacturer Part Number" "CRCW060310K0FKEA"
+		(property "Manufacturer Part Number" "RC0603FR-0710KL"
 			(at 123.19 69.85 0)
 			(effects
@@
 			)
 		)
-		(property "Mouser Part Number" "71-CRCW0603-10K-E3"
+		(property "Mouser Part Number" "603-RC0603FR-0710KL"
+			(at 123.19 69.85 0)
+			(effects
+				(font
+					(size 1.27 1.27)
+				)
+				(hide yes)
+			)
+		)
+		(property "Ullmanna Part Number" "BMCR0201"
 			(at 123.19 69.85 0)
 			(effects
@@
 			(at 86.36 52.07 0)
 			(effects
+				(font
+					(size 1.27 1.27)
+				)
+				(hide yes)
+			)
+		)
+		(property "Ullmanna Part Number" ""
+			(at 86.36 52.07 0)
+			(effects
