File: kicad/Impact_driver_controller/Drivers.kicad_sch (KiCad schematic)
At the start: 19 parts, among them U1 DRV8874_module, U4 DRV8874_module, U5 DRV8874_module, U7 DRV8874_module, U8 DRV8874_module, U9 DRV8874_module

Commit message: Connector for bigger current, control module 2
Parts:
- D1, D3, D5, D6, D7, D8: Mouser Part Number (none) -> 78-VLMS1300-GS08
- R10, R5, R6, R7, R8, R9: Mouser Part Number (none) -> 71-CRCW0603-1.0K-E3
- RV1: Mouser Part Number (none) -> 652-3296W-1-104LF

Commit message: Add part numbers
Parts:
- D1, D3, D5, D6, D7, D8: Manufacturer Part Number (none) -> VLMS1300-GS08
- R10, R5, R6, R7, R8, R9: Manufacturer Part Number (none) -> CRCW06031K00FKEA
- RV1: value W203 (100K) -> 100k; Manufacturer Part Number (none) -> 3296W-1-104LF
Changed lines of the file:
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@@
 			)
 		)
-		(property "Value" "W203 (100K)"
+		(property "Value" "100k"
 			(at 154.94 40.6399 0)
 			(effects
@@
 			)
 		)
-		(property "Description" ""
+		(property "Description" "CUSTOM"
 			(at 157.48 39.37 0)
 			(effects
@@
 			)
 		)
-		(property "Manufacturer Part Number" ""
+		(property "Manufacturer Part Number" "3296W-1-104LF"
 			(at 157.48 39.37 0)
 			(effects
@@
 			)
 		)
-		(property "Description" ""
+		(property "Description" "ULM"
 			(at 201.93 36.83 0)
 			(effects
@@
 			)
 		)
-		(property "Manufacturer Part Number" ""
+		(property "Manufacturer Part Number" "CRCW06031K00FKEA"
 			(at 201.93 36.83 0)
 			(effects
@@
 			)
 		)
-		(property "Description" ""
+		(property "Description" "ULM"
 			(at 210.82 36.83 0)
 			(effects
@@
 			)
 		)
-		(property "Manufacturer Part Number" ""
+		(property "Manufacturer Part Number" "CRCW06031K00FKEA"
 			(at 210.82 36.83 0)
 			(effects
@@
 			)
 		)
-		(property "Description" ""
+		(property "Description" "ULM"
 			(at 191.77 36.83 0)
 			(effects
@@
 			)
 		)
-		(property "Manufacturer Part Number" ""
+		(property "Manufacturer Part Number" "CRCW06031K00FKEA"
 			(at 191.77 36.83 0)
 			(effects
@@
 			)
 		)
-		(property "Description" ""
+		(property "Description" "ULM"
 			(at 210.82 44.45 0)
 			(effects
@@
 			)
 		)
-		(property "Manufacturer Part Number" ""
+		(property "Manufacturer Part Number" "VLMS1300-GS08"
 			(at 210.82 44.45 0)
 			(effects
@@
 			)
 		)
-		(property "Description" ""
+		(property "Description" "ULM"
 			(at 191.77 44.45 0)
 			(effects
@@
 			)
 		)
-		(property "Manufacturer Part Number" ""
+		(property "Manufacturer Part Number" "VLMS1300-GS08"
 			(at 191.77 44.45 0)
 			(effects
@@
 			)
 		)
-		(property "Description" ""
+		(property "Description" "ULM"
 			(at 219.71 36.83 0)
 			(effects
@@
 			)
 		)
-		(property "Manufacturer Part Number" ""
+		(property "Manufacturer Part Number" "CRCW06031K00FKEA"
 			(at 219.71 36.83 0)
 			(effects
@@
 			)
 		)
-		(property "Description" ""
+		(property "Description" "ULM"
 			(at 181.61 36.83 0)
 			(effects
@@
 			)
 		)
-		(property "Manufacturer Part Number" ""
+		(property "Manufacturer Part Number" "CRCW06031K00FKEA"
 			(at 181.61 36.83 0)
 			(effects
@@
 			)
 		)
-		(property "Description" ""
+		(property "Description" "ULM"
 			(at 181.61 44.45 0)
 			(effects
@@
 			)
 		)
-		(property "Manufacturer Part Number" ""
+		(property "Manufacturer Part Number" "VLMS1300-GS08"
 			(at 181.61 44.45 0)
 			(effects
@@
 			)
 		)
-		(property "Description" ""
+		(property "Description" "ULM"
 			(at 219.71 44.45 0)
 			(effects
@@
 			)
 		)
-		(property "Manufacturer Part Number" ""
+		(property "Manufacturer Part Number" "VLMS1300-GS08"
 			(at 219.71 44.45 0)
 			(effects
@@
 			)
 		)
-		(property "Description" ""
+		(property "Description" "ULM"
 			(at 201.93 44.45 0)
 			(effects
@@
 			)
 		)
-		(property "Manufacturer Part Number" ""
+		(property "Manufacturer Part Number" "VLMS1300-GS08"
 			(at 201.93 44.45 0)
 			(effects
@@
 			)
 		)
-		(property "Description" ""
+		(property "Description" "ULM"
 			(at 228.6 44.45 0)
 			(effects
@@
 			)
 		)
-		(property "Manufacturer Part Number" ""
+		(property "Manufacturer Part Number" "VLMS1300-GS08"
 			(at 228.6 44.45 0)
 			(effects
@@
 			)
 		)
-		(property "Description" ""
+		(property "Description" "ULM"
 			(at 228.6 36.83 0)
 			(effects
@@
 			)
 		)
-		(property "Manufacturer Part Number" ""
+		(property "Manufacturer Part Number" "CRCW06031K00FKEA"
 			(at 228.6 36.83 0)
 			(effects

Commit message: BOM with Ullmanna part numbers
Parts:
- D1, D3, D5, D6, D7, D8: Manufacturer Part Number VLMS1300-GS08 -> APTD1608LSURCK; Mouser Part Number 78-VLMS1300-GS08 -> 604-APTD1608LSURCK; Ullmanna Part Number (none) -> BMCLED004
- R10, R5, R6, R7, R8, R9: Manufacturer Part Number CRCW06031K00FKEA -> RC0603FR-071KL; Mouser Part Number 71-CRCW0603-1.0K-E3 -> 603-RC0603FR-071KL; Ullmanna Part Number (none) -> BMCR0176

Commit message: LED footprint update
Parts:
- D1, D3, D5, D6, D7, D8: footprint LED_SMD:LED_0603_1608Metric_Pad1.05x0.95mm_HandSolder -> LED_SMD:LED_0805_2012Metric_Pad1.15x1.40mm_HandSolder; Manufacturer Part Number APTD1608LSURCK -> APTD2012LSURCK; Mouser Part Number 604-APTD1608LSURCK -> 604-APTD2012LSURCK; Ullmanna Part Number BMCLED004 -> BMCLED104
Changed lines of the file:
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@@
 			)
 		)
-		(property "Footprint" "LED_SMD:LED_0603_1608Metric_Pad1.05x0.95mm_HandSolder"
+		(property "Footprint" "LED_SMD:LED_0805_2012Metric_Pad1.15x1.40mm_HandSolder"
 			(at 210.82 44.45 0)
 			(effects
@@
 			)
 		)
-		(property "Manufacturer Part Number" "APTD1608LSURCK"
+		(property "Manufacturer Part Number" "APTD2012LSURCK "
 			(at 210.82 44.45 0)
 			(effects
@@
 			)
 		)
-		(property "Mouser Part Number" "604-APTD1608LSURCK"
+		(property "Mouser Part Number" "604-APTD2012LSURCK "
 			(at 210.82 44.45 0)
 			(effects
@@
 			)
 		)
-		(property "Ullmanna Part Number" "BMCLED004"
+		(property "Ullmanna Part Number" "BMCLED104 "
 			(at 210.82 44.45 0)
 			(effects
@@
 			)
 		)
-		(property "Footprint" "LED_SMD:LED_0603_1608Metric_Pad1.05x0.95mm_HandSolder"
+		(property "Footprint" "LED_SMD:LED_0805_2012Metric_Pad1.15x1.40mm_HandSolder"
 			(at 191.77 44.45 0)
 			(effects
@@
 			)
 		)
-		(property "Manufacturer Part Number" "APTD1608LSURCK"
+		(property "Manufacturer Part Number" "APTD2012LSURCK "
 			(at 191.77 44.45 0)
 			(effects
@@
 			)
 		)
-		(property "Mouser Part Number" "604-APTD1608LSURCK"
+		(property "Mouser Part Number" "604-APTD2012LSURCK "
 			(at 191.77 44.45 0)
 			(effects
@@
 			)
 		)
-		(property "Ullmanna Part Number" "BMCLED004"
+		(property "Ullmanna Part Number" "BMCLED104 "
 			(at 191.77 44.45 0)
 			(effects
@@
 			)
 		)
-		(property "Footprint" "LED_SMD:LED_0603_1608Metric_Pad1.05x0.95mm_HandSolder"
+		(property "Footprint" "LED_SMD:LED_0805_2012Metric_Pad1.15x1.40mm_HandSolder"
 			(at 181.61 44.45 0)
 			(effects
@@
 			)
 		)
-		(property "Manufacturer Part Number" "APTD1608LSURCK"
+		(property "Manufacturer Part Number" "APTD2012LSURCK "
 			(at 181.61 44.45 0)
 			(effects
@@
 			)
 		)
-		(property "Mouser Part Number" "604-APTD1608LSURCK"
+		(property "Mouser Part Number" "604-APTD2012LSURCK "
 			(at 181.61 44.45 0)
 			(effects
@@
 			)
 		)
-		(property "Ullmanna Part Number" "BMCLED004"
+		(property "Ullmanna Part Number" "BMCLED104 "
 			(at 181.61 44.45 0)
 			(effects
@@
 			)
 		)
-		(property "Footprint" "LED_SMD:LED_0603_1608Metric_Pad1.05x0.95mm_HandSolder"
+		(property "Footprint" "LED_SMD:LED_0805_2012Metric_Pad1.15x1.40mm_HandSolder"
 			(at 219.71 44.45 0)
 			(effects
@@
 			)
 		)
-		(property "Manufacturer Part Number" "APTD1608LSURCK"
+		(property "Manufacturer Part Number" "APTD2012LSURCK "
 			(at 219.71 44.45 0)
 			(effects
@@
 			)
 		)
-		(property "Mouser Part Number" "604-APTD1608LSURCK"
+		(property "Mouser Part Number" "604-APTD2012LSURCK "
 			(at 219.71 44.45 0)
 			(effects
@@
 			)
 		)
-		(property "Ullmanna Part Number" "BMCLED004"
+		(property "Ullmanna Part Number" "BMCLED104 "
 			(at 219.71 44.45 0)
 			(effects
@@
 			)
 		)
-		(property "Footprint" "LED_SMD:LED_0603_1608Metric_Pad1.05x0.95mm_HandSolder"
+		(property "Footprint" "LED_SMD:LED_0805_2012Metric_Pad1.15x1.40mm_HandSolder"
 			(at 201.93 44.45 0)
 			(effects
@@
 			)
 		)
-		(property "Manufacturer Part Number" "APTD1608LSURCK"
+		(property "Manufacturer Part Number" "APTD2012LSURCK "
 			(at 201.93 44.45 0)
 			(effects
@@
 			)
 		)
-		(property "Mouser Part Number" "604-APTD1608LSURCK"
+		(property "Mouser Part Number" "604-APTD2012LSURCK "
 			(at 201.93 44.45 0)
 			(effects
@@
 			)
 		)
-		(property "Ullmanna Part Number" "BMCLED004"
+		(property "Ullmanna Part Number" "BMCLED104 "
 			(at 201.93 44.45 0)
 			(effects
@@
 			)
 		)
-		(property "Footprint" "LED_SMD:LED_0603_1608Metric_Pad1.05x0.95mm_HandSolder"
+		(property "Footprint" "LED_SMD:LED_0805_2012Metric_Pad1.15x1.40mm_HandSolder"
 			(at 228.6 44.45 0)
 			(effects
@@
 			)
 		)
-		(property "Manufacturer Part Number" "APTD1608LSURCK"
+		(property "Manufacturer Part Number" "APTD2012LSURCK "
 			(at 228.6 44.45 0)
 			(effects
@@
 			)
 		)
-		(property "Mouser Part Number" "604-APTD1608LSURCK"
+		(property "Mouser Part Number" "604-APTD2012LSURCK "
 			(at 228.6 44.45 0)
 			(effects
@@
 			)
 		)
-		(property "Ullmanna Part Number" "BMCLED004"
+		(property "Ullmanna Part Number" "BMCLED104 "
 			(at 228.6 44.45 0)
 			(effects
