File: kicad/Impact_driver_controller/power_supply.kicad_sch (KiCad schematic)
At the start: 11 parts, among them U3 LM78M05, U4 LM78M12

Commit message: Main board schematic
Parts:
- removed C12: 0.1 uF, Capacitor_SMD:C_1206_3216Metric_Pad1.33x1.80mm_HandSolder, symbol Device:C
- removed C6: 100uF, Capacitor_SMD:CP_Elec_8x10, symbol Device:C_Polarized
- removed C8: 0.33 uF, Capacitor_SMD:C_1206_3216Metric_Pad1.33x1.80mm_HandSolder, symbol Device:C
- removed D3: SS34A, Diode_SMD:D_SMB-SMC_Universal_Handsoldering, symbol Device:D_Schottky
- removed F2: 1A, Fuse:Fuse_Blade_ATO_directSolder, symbol Device:Fuse
- removed U4: LM78M12, Package_TO_SOT_SMD:TO-252-2, symbol Regulator_Linear:LM7812_TO220
- added C1: 100 uF, 25V, Capacitor_Tantalum_SMD:CP_EIA-7343-40_Kemet-Y_Pad2.25x2.55mm_HandSolder, symbol Device:C_Polarized
- added D2: SS34, Diode_SMD:D_SMB-SMC_Universal_Handsoldering, symbol Device:D_Schottky
- added F1: 1 A, Fuse:Fuseholder_Blade_Mini_Keystone_3568, symbol Device:Fuse
- C7: value 0.33 uF -> 0.47uF
- C9: value 0.1 uF -> 0.1uF; footprint Capacitor_SMD:C_1206_3216Metric_Pad1.33x1.80mm_HandSolder -> Capacitor_SMD:C_0603_1608Metric_Pad1.08x0.95mm_HandSolder
- D4: value LED -> LED_GREEN; footprint Diode_SMD:D_1206_3216Metric_Pad1.42x1.75mm_HandSolder -> LED_SMD:LED_0603_1608Metric_Pad1.05x0.95mm_HandSolder
Connections:
- net GND: now also C1.2
- net +12V: no longer names the net of C7.1, U3.1 (VI)
- net +12V: now also C1.1, F1.1
- new net: D2.1 (K), F1.2
- new net +VDD_OUT: D2.2 (A)
Other:
- moved on the sheet: C7, C9, D4, R4, U3

Commit message: First main board layout
Parts:
- R4: footprint Resistor_SMD:R_1206_3216Metric_Pad1.30x1.75mm_HandSolder -> Resistor_SMD:R_0603_1608Metric_Pad0.98x0.95mm_HandSolder
Changed lines of the file:
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@@
 			)
 		)
-		(property "Footprint" "Resistor_SMD:R_1206_3216Metric_Pad1.30x1.75mm_HandSolder"
+		(property "Footprint" "Resistor_SMD:R_0603_1608Metric_Pad0.98x0.95mm_HandSolder"
 			(at 127 68.072 90)
 			(effects

Commit message: Connector for bigger current, control module 2
Parts:
- C1: Mouser Part Number (none) -> 80-T491X107M25ATAUTO
- C7: Mouser Part Number (none) -> 80-C1206C474K5RAULR
- C9: Mouser Part Number (none) -> 80-C0603C104K5RAUTO
- D2: Mouser Part Number (none) -> 512-SS34
- D4: Mouser Part Number (none) -> 78-VLMG1300-GS08
- F1: Mouser Part Number (none) -> 534-3568
- R4: Mouser Part Number (none) -> 71-CRCW0603-1.0K-E3
- U3: Mouser Part Number (none) -> 511-L78M05CDT-TR
Changed lines of the file:
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@@
 			)
 		)
-		(property "Description" "78-VLMG1300-GS08"
+		(property "Description" ""
+			(at 134.62 74.93 0)
+			(effects
+				(font
+					(size 1.27 1.27)
+				)
+				(hide yes)
+			)
+		)
+		(property "Manufacturer Part Number" ""
+			(at 134.62 74.93 0)
+			(effects
+				(font
+					(size 1.27 1.27)
+				)
+				(hide yes)
+			)
+		)
+		(property "Mouser Part Number" "78-VLMG1300-GS08"
 			(at 134.62 74.93 0)
 			(effects
@@
 			)
 		)
-		(property "Description" "512-SS34"
+		(property "Description" ""
+			(at 74.93 54.61 0)
+			(effects
+				(font
+					(size 1.27 1.27)
+				)
+				(hide yes)
+			)
+		)
+		(property "Manufacturer Part Number" ""
+			(at 74.93 54.61 0)
+			(effects
+				(font
+					(size 1.27 1.27)
+				)
+				(hide yes)
+			)
+		)
+		(property "Mouser Part Number" "512-SS34"
 			(at 74.93 54.61 0)
 			(effects
@@
 			)
 		)
-		(property "Description" "80-T491X107M25ATAUTO"
+		(property "Description" ""
+			(at 74.93 76.2 0)
+			(effects
+				(font
+					(size 1.27 1.27)
+				)
+				(hide yes)
+			)
+		)
+		(property "Manufacturer Part Number" ""
+			(at 74.93 76.2 0)
+			(effects
+				(font
+					(size 1.27 1.27)
+				)
+				(hide yes)
+			)
+		)
+		(property "Mouser Part Number" "80-T491X107M25ATAUTO"
 			(at 74.93 76.2 0)
 			(effects
@@
 			)
 		)
-		(property "Description" "534-3568"
+		(property "Description" ""
+			(at 74.93 63.5 0)
+			(effects
+				(font
+					(size 1.27 1.27)
+				)
+				(hide yes)
+			)
+		)
+		(property "Manufacturer Part Number" ""
+			(at 74.93 63.5 0)
+			(effects
+				(font
+					(size 1.27 1.27)
+				)
+				(hide yes)
+			)
+		)
+		(property "Mouser Part Number" "534-3568"
 			(at 74.93 63.5 0)
 			(effects
@@
 			)
 		)
-		(property "Description" "71-CRCW0603-1.0K-E3"
+		(property "Description" ""
+			(at 127 69.85 0)
+			(effects
+				(font
+					(size 1.27 1.27)
+				)
+				(hide yes)
+			)
+		)
+		(property "Manufacturer Part Number" ""
+			(at 127 69.85 0)
+			(effects
+				(font
+					(size 1.27 1.27)
+				)
+				(hide yes)
+			)
+		)
+		(property "Mouser Part Number" "71-CRCW0603-1.0K-E3"
 			(at 127 69.85 0)
 			(effects
@@
 			)
 		)
-		(property "Description" "80-C1206C474K5RAULR"
+		(property "Description" ""
+			(at 88.9 76.2 0)
+			(effects
+				(font
+					(size 1.27 1.27)
+				)
+				(hide yes)
+			)
+		)
+		(property "Manufacturer Part Number" ""
+			(at 88.9 76.2 0)
+			(effects
+				(font
+					(size 1.27 1.27)
+				)
+				(hide yes)
+			)
+		)
+		(property "Mouser Part Number" "80-C1206C474K5RAULR"
 			(at 88.9 76.2 0)
 			(effects
@@
 			)
 		)
-		(property "Description" "511-L78M05CDT-TR"
+		(property "Description" ""
+			(at 104.14 69.85 0)
+			(effects
+				(font
+					(size 1.27 1.27)
+				)
+				(hide yes)
+			)
+		)
+		(property "Manufacturer Part Number" ""
+			(at 104.14 69.85 0)
+			(effects
+				(font
+					(size 1.27 1.27)
+				)
+				(hide yes)
+			)
+		)
+		(property "Mouser Part Number" "511-L78M05CDT-TR"
 			(at 104.14 69.85 0)
 			(effects
@@
 			)
 		)
-		(property "Description" "80-C0603C104K5RAUTO"
+		(property "Description" ""
 			(at 118.11 76.2 0)
 			(effects
+				(font
+					(size 1.27 1.27)
+				)
+				(hide yes)
+			)
+		)
+		(property "Manufacturer Part Number" ""
+			(at 118.11 76.2 0)
+			(effects
+				(font
+					(size 1.27 1.27)
+				)
+				(hide yes)
+			)
+		)
+		(property "Mouser Part Number" "80-C0603C104K5RAUTO"
+			(at 118.11 76.2 0)
+			(effects

Commit message: Add part numbers
Parts:
- C1: value 100 uF, 25V -> 100uF; Manufacturer Part Number (none) -> T491X107M025ATAUTO
- C7: Manufacturer Part Number (none) -> C1206C474K5RACAUTO7210
- C9: Manufacturer Part Number (none) -> C0603C104K5RACAUTO
- D2: Manufacturer Part Number (none) -> SS34
- D4: Manufacturer Part Number (none) -> VLMG1300-GS08
- F1: value 1 A -> FUSE 1A; Manufacturer Part Number (none) -> 3568
- R4: Manufacturer Part Number (none) -> CRCW06031K00FKEA
- U3: Manufacturer Part Number (none) -> L78M05CDT-TR
Changed lines of the file:
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@@
 			)
 		)
-		(property "Description" ""
+		(property "Description" "ULM"
 			(at 134.62 74.93 0)
 			(effects
@@
 			)
 		)
-		(property "Manufacturer Part Number" ""
+		(property "Manufacturer Part Number" "VLMG1300-GS08"
 			(at 134.62 74.93 0)
 			(effects
@@
 			)
 		)
-		(property "Description" ""
+		(property "Description" "CUSTOM"
 			(at 74.93 54.61 0)
 			(effects
@@
 			)
 		)
-		(property "Manufacturer Part Number" ""
+		(property "Manufacturer Part Number" "SS34"
 			(at 74.93 54.61 0)
 			(effects
@@
 			)
 		)
-		(property "Value" "100 uF, 25V"
+		(property "Value" "100uF"
 			(at 71.374 82.55 90)
 			(effects
@@
 			)
 		)
-		(property "Description" ""
+		(property "Description" "ULM"
 			(at 74.93 76.2 0)
 			(effects
@@
 			)
 		)
-		(property "Manufacturer Part Number" ""
+		(property "Manufacturer Part Number" "T491X107M025ATAUTO"
 			(at 74.93 76.2 0)
 			(effects
@@
 			)
 		)
-		(property "Value" "1 A"
+		(property "Value" "FUSE 1A"
 			(at 77.47 64.7699 0)
 			(effects
@@
 			)
 		)
-		(property "Description" ""
+		(property "Description" "ULM"
 			(at 74.93 63.5 0)
 			(effects
@@
 			)
 		)
-		(property "Manufacturer Part Number" ""
+		(property "Manufacturer Part Number" "3568"
 			(at 74.93 63.5 0)
 			(effects
@@
 			)
 		)
-		(property "Description" ""
+		(property "Description" "ULM"
 			(at 127 69.85 0)
 			(effects
@@
 			)
 		)
-		(property "Manufacturer Part Number" ""
+		(property "Manufacturer Part Number" "CRCW06031K00FKEA"
 			(at 127 69.85 0)
 			(effects
@@
 			)
 		)
-		(property "Description" ""
+		(property "Description" "ULM"
 			(at 88.9 76.2 0)
 			(effects
@@
 			)
 		)
-		(property "Manufacturer Part Number" ""
+		(property "Manufacturer Part Number" "C1206C474K5RACAUTO7210"
 			(at 88.9 76.2 0)
 			(effects
@@
 			)
 		)
-		(property "Description" ""
+		(property "Description" "CUSTOM"
 			(at 104.14 69.85 0)
 			(effects
@@
 			)
 		)
-		(property "Manufacturer Part Number" ""
+		(property "Manufacturer Part Number" "L78M05CDT-TR"
 			(at 104.14 69.85 0)
 			(effects
@@
 			)
 		)
-		(property "Description" ""
+		(property "Description" "ULM"
 			(at 118.11 76.2 0)
 			(effects
@@
 			)
 		)
-		(property "Manufacturer Part Number" ""
+		(property "Manufacturer Part Number" "C0603C104K5RACAUTO"
 			(at 118.11 76.2 0)
 			(effects

Commit message: BOM with Ullmanna part numbers
Parts:
- C7: Manufacturer Part Number C1206C474K5RACAUTO7210 -> C1608X5R1C475KE; Mouser Part Number 80-C1206C474K5RAULR -> 810-C1608X5R1C475KE; Ullmanna Part Number (none) -> BMCCK404
- C9: Manufacturer Part Number C0603C104K5RACAUTO -> C0603C104M5RACTU; Mouser Part Number 80-C0603C104K5RAUTO -> 80-C0603C104M5R; Ullmanna Part Number (none) -> BMCCK351
- D4: Manufacturer Part Number VLMG1300-GS08 -> APTD1608LCGCK; Mouser Part Number 78-VLMG1300-GS08 -> 604-APTD1608LCGCK; Ullmanna Part Number (none) -> BMCLED002
- R4: Manufacturer Part Number CRCW06031K00FKEA -> RC0603FR-071KL; Mouser Part Number 71-CRCW0603-1.0K-E3 -> 603-RC0603FR-071KL; Ullmanna Part Number (none) -> BMCR0176
Changed lines of the file:
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@@
 (kicad_sch
-	(version 20231120)
+	(version 20250114)
 	(generator "eeschema")
-	(generator_version "8.0")
+	(generator_version "9.0")
 	(paper "A5")
 	(junction
@@
 		(shape output)
 		(at 62.23 52.07 270)
-		(fields_autoplaced yes)
 		(effects
 			(font
@@
 		(shape output)
 		(at 62.23 40.64 0)
-		(fields_autoplaced yes)
 		(effects
 			(font
@@
 		(shape input)
 		(at 62.23 44.45 0)
-		(fields_autoplaced yes)
 		(effects
 			(font
@@
 		(shape input)
 		(at 58.42 31.75 180)
-		(fields_autoplaced yes)
 		(effects
 			(font
@@
 			)
 		)
-		(property "Manufacturer Part Number" "VLMG1300-GS08"
+		(property "Manufacturer Part Number" "APTD1608LCGCK "
 			(at 134.62 74.93 0)
 			(effects
@@
 			)
 		)
-		(property "Mouser Part Number" "78-VLMG1300-GS08"
+		(property "Mouser Part Number" "604-APTD1608LCGCK "
 			(at 134.62 74.93 0)
+			(effects
+				(font
+					(size 1.27 1.27)
+				)
+				(hide yes)
+			)
+		)
+		(property "Ullmanna Part Number" "BMCLED002 "
+			(at 134.62 74.93 90)
 			(effects
 				(font
@@
 			)
 		)
+		(property "Ullmanna Part Number" ""
+			(at 74.93 54.61 90)
+			(effects
+				(font
+					(size 1.27 1.27)
+				)
+				(hide yes)
+			)
+		)
 		(pin "1"
 		)
@@
 			)
 		)
-		(property "Description" "ULM"
+		(property "Description" "ADD"
 			(at 74.93 76.2 0)
 			(effects
@@
 		(property "Mouser Part Number" "80-T491X107M25ATAUTO"
 			(at 74.93 76.2 0)
+			(effects
+				(font
+					(size 1.27 1.27)
+				)
+				(hide yes)
+			)
+		)
+		(property "Ullmanna Part Number" "~"
+			(at 74.93 76.2 90)
 			(effects
 				(font
@@
 			)
 		)
+		(property "Ullmanna Part Number" "~"
+			(at 74.93 63.5 0)
+			(effects
+				(font
+					(size 1.27 1.27)
+				)
+				(hide yes)
+			)
+		)
 		(pin "1"
 		)
@@
 			)
 		)
-		(property "Manufacturer Part Number" "CRCW06031K00FKEA"
+		(property "Manufacturer Part Number" "RC0603FR-071KL"
 			(at 127 69.85 0)
 			(effects
@@
 			)
 		)
-		(property "Mouser Part Number" "71-CRCW0603-1.0K-E3"
+		(property "Mouser Part Number" "603-RC0603FR-071KL"
 			(at 127 69.85 0)
+			(effects
+				(font
+					(size 1.27 1.27)
+				)
+				(hide yes)
+			)
+		)
+		(property "Ullmanna Part Number" "BMCR0176 "
+			(at 127 69.85 90)
 			(effects
 				(font
@@
 			)
 		)
-		(property "Manufacturer Part Number" "C1206C474K5RACAUTO7210"
+		(property "Manufacturer Part Number" "C1608X5R1C475KE"
 			(at 88.9 76.2 0)
 			(effects
@@
 			)
 		)
-		(property "Mouser Part Number" "80-C1206C474K5RAULR"
+		(property "Mouser Part Number" "810-C1608X5R1C475KE"
+			(at 88.9 76.2 0)
+			(effects
+				(font
+					(size 1.27 1.27)
+				)
+				(hide yes)
+			)
+		)
+		(property "Ullmanna Part Number" "BMCCK404"
 			(at 88.9 76.2 0)
 			(effects
@@
 			)
 		)
+		(property "Ullmanna Part Number" ""
+			(at 104.14 69.85 0)
+			(effects
+				(font
+					(size 1.27 1.27)
+				)
+				(hide yes)
+			)
+		)
 		(pin "3"
 		)
@@
 			)
 		)
-		(property "Manufacturer Part Number" "C0603C104K5RACAUTO"
+		(property "Manufacturer Part Number" "C0603C104M5RACTU"
 			(at 118.11 76.2 0)
 			(effects
@@
 			)
 		)
-		(property "Mouser Part Number" "80-C0603C104K5RAUTO"
+		(property "Mouser Part Number" "80-C0603C104M5R"
 			(at 118.11 76.2 0)
 			(effects
+				(font
+					(size 1.27 1.27)
+				)
+				(hide yes)
+			)
+		)
+		(property "Ullmanna Part Number" "BMCCK351"
+			(at 118.11 76.2 0)
+			(effects

Commit message: LED footprint update
Parts:
- D4: footprint LED_SMD:LED_0603_1608Metric_Pad1.05x0.95mm_HandSolder -> LED_SMD:LED_0805_2012Metric_Pad1.15x1.40mm_HandSolder; Manufacturer Part Number APTD1608LCGCK -> APTD2012LCGCK; Mouser Part Number 604-APTD1608LCGCK -> 604-APTD2012LCGCK; Ullmanna Part Number BMCLED002 -> BMCLED102
Changed lines of the file:
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@@
 			)
 		)
-		(property "Footprint" "LED_SMD:LED_0603_1608Metric_Pad1.05x0.95mm_HandSolder"
+		(property "Footprint" "LED_SMD:LED_0805_2012Metric_Pad1.15x1.40mm_HandSolder"
 			(at 134.62 74.93 0)
 			(effects
@@
 			)
 		)
-		(property "Manufacturer Part Number" "APTD1608LCGCK "
+		(property "Manufacturer Part Number" "APTD2012LCGCK "
 			(at 134.62 74.93 0)
 			(effects
@@
 			)
 		)
-		(property "Mouser Part Number" "604-APTD1608LCGCK "
+		(property "Mouser Part Number" "604-APTD2012LCGCK "
 			(at 134.62 74.93 0)
 			(effects
@@
 			)
 		)
-		(property "Ullmanna Part Number" "BMCLED002 "
+		(property "Ullmanna Part Number" "BMCLED102 "
 			(at 134.62 74.93 90)
 			(effects
