File: kicad/modules/MCU_module/filters.kicad_sch (KiCad schematic)
At the start: 6 parts

Commit message: Connector for bigger current, control module 2
Parts:
- C1: Mouser number (none) -> 77-VJ0603Y332KXBAC
- C2, C3: Mouser number (none) -> 80-C1206C105K5RAUTO
- R1, R2, R3: Mouser number (none) -> 71-CRCW0603-10K-E3
Changed lines of the file:
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@@
 			)
 		)
-		(property "Description" "71-CRCW0603-10K-E3"
+		(property "Description" ""
+			(at 96.52 29.21 0)
+			(effects
+				(font
+					(size 1.27 1.27)
+				)
+				(hide yes)
+			)
+		)
+		(property "Manufacturer Part Number" ""
+			(at 96.52 29.21 0)
+			(effects
+				(font
+					(size 1.27 1.27)
+				)
+				(hide yes)
+			)
+		)
+		(property "Mouser number" "71-CRCW0603-10K-E3"
 			(at 96.52 29.21 0)
 			(effects
@@
 			)
 		)
-		(property "Description" "80-C1206C105K5RAUTO"
+		(property "Description" ""
+			(at 106.68 34.29 0)
+			(effects
+				(font
+					(size 1.27 1.27)
+				)
+				(hide yes)
+			)
+		)
+		(property "Manufacturer Part Number" ""
+			(at 106.68 34.29 0)
+			(effects
+				(font
+					(size 1.27 1.27)
+				)
+				(hide yes)
+			)
+		)
+		(property "Mouser number" "80-C1206C105K5RAUTO"
 			(at 106.68 34.29 0)
 			(effects
@@
 			)
 		)
-		(property "Description" "71-CRCW0603-10K-E3"
+		(property "Description" ""
+			(at 96.52 77.47 0)
+			(effects
+				(font
+					(size 1.27 1.27)
+				)
+				(hide yes)
+			)
+		)
+		(property "Manufacturer Part Number" ""
+			(at 96.52 77.47 0)
+			(effects
+				(font
+					(size 1.27 1.27)
+				)
+				(hide yes)
+			)
+		)
+		(property "Mouser number" "71-CRCW0603-10K-E3"
 			(at 96.52 77.47 0)
 			(effects
@@
 			)
 		)
-		(property "Description" "Unpolarized capacitor"
+		(property "Description" ""
+			(at 106.68 58.42 0)
+			(effects
+				(font
+					(size 1.27 1.27)
+				)
+				(hide yes)
+			)
+		)
+		(property "Manufacturer Part Number" ""
+			(at 106.68 58.42 0)
+			(effects
+				(font
+					(size 1.27 1.27)
+				)
+				(hide yes)
+			)
+		)
+		(property "Mouser number" "77-VJ0603Y332KXBAC"
 			(at 106.68 58.42 0)
 			(effects
@@
 			)
 		)
-		(property "Description" "71-CRCW0603-10K-E3"
+		(property "Description" ""
+			(at 96.52 53.34 0)
+			(effects
+				(font
+					(size 1.27 1.27)
+				)
+				(hide yes)
+			)
+		)
+		(property "Manufacturer Part Number" ""
+			(at 96.52 53.34 0)
+			(effects
+				(font
+					(size 1.27 1.27)
+				)
+				(hide yes)
+			)
+		)
+		(property "Mouser number" "71-CRCW0603-10K-E3"
 			(at 96.52 53.34 0)
 			(effects
@@
 			)
 		)
-		(property "Description" "80-C1206C105K5RAUTO"
+		(property "Description" ""
 			(at 106.68 82.55 0)
 			(effects
+				(font
+					(size 1.27 1.27)
+				)
+				(hide yes)
+			)
+		)
+		(property "Manufacturer Part Number" ""
+			(at 106.68 82.55 0)
+			(effects
+				(font
+					(size 1.27 1.27)
+				)
+				(hide yes)
+			)
+		)
+		(property "Mouser number" "80-C1206C105K5RAUTO"
+			(at 106.68 82.55 0)
+			(effects

Commit message: Add part numbers
Parts:
- C1: value 3.3 nF -> 3.3nF; Manufacturer Part Number (none) -> VJ0603Y332KXBAC
- C2: value 1 uF -> 1uF; Manufacturer Part Number (none) -> C1206C105K5RACAUTO
- C3: value none -> 1uF; Manufacturer Part Number (none) -> C1206C105K5RACAUTO
- R1, R2: footprint Capacitor_SMD:C_0603_1608Metric_Pad1.08x0.95mm_HandSolder -> Resistor_SMD:R_0603_1608Metric_Pad0.98x0.95mm_HandSolder; Manufacturer Part Number (none) -> CRCW060310K0FKEA
- R3: value none -> 10k; footprint Capacitor_SMD:C_0603_1608Metric_Pad1.08x0.95mm_HandSolder -> Resistor_SMD:R_0603_1608Metric_Pad0.98x0.95mm_HandSolder; Manufacturer Part Number (none) -> CRCW060310K0FKEA
Changed lines of the file:
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@@
 			)
 		)
-		(property "Value" "none"
+		(property "Value" "10k"
 			(at 96.52 26.924 90)
 			(effects
@@
 			)
 		)
-		(property "Footprint" "Capacitor_SMD:C_0603_1608Metric_Pad1.08x0.95mm_HandSolder"
+		(property "Footprint" "Resistor_SMD:R_0603_1608Metric_Pad0.98x0.95mm_HandSolder"
 			(at 96.52 27.432 90)
 			(effects
@@
 			)
 		)
-		(property "Description" ""
+		(property "Description" "ULM"
 			(at 96.52 29.21 0)
 			(effects
@@
 			)
 		)
-		(property "Manufacturer Part Number" ""
+		(property "Manufacturer Part Number" "CRCW060310K0FKEA"
 			(at 96.52 29.21 0)
 			(effects
@@
 			)
 		)
-		(property "Value" "none"
+		(property "Value" "1uF"
 			(at 110.49 35.5599 0)
 			(effects
@@
 			)
 		)
-		(property "Description" ""
+		(property "Description" "ULM"
 			(at 106.68 34.29 0)
 			(effects
@@
 			)
 		)
-		(property "Manufacturer Part Number" ""
+		(property "Manufacturer Part Number" "C1206C105K5RACAUTO"
 			(at 106.68 34.29 0)
 			(effects
@@
 			)
 		)
-		(property "Footprint" "Capacitor_SMD:C_0603_1608Metric_Pad1.08x0.95mm_HandSolder"
+		(property "Footprint" "Resistor_SMD:R_0603_1608Metric_Pad0.98x0.95mm_HandSolder"
 			(at 96.52 75.692 90)
 			(effects
@@
 			)
 		)
-		(property "Description" ""
+		(property "Description" "ULM"
 			(at 96.52 77.47 0)
 			(effects
@@
 			)
 		)
-		(property "Manufacturer Part Number" ""
+		(property "Manufacturer Part Number" "CRCW060310K0FKEA"
 			(at 96.52 77.47 0)
 			(effects
@@
 			)
 		)
-		(property "Value" "3.3 nF"
+		(property "Value" "3.3nF"
 			(at 110.49 59.6899 0)
 			(effects
@@
 			)
 		)
-		(property "Description" ""
+		(property "Description" "CUSTOM"
 			(at 106.68 58.42 0)
 			(effects
@@
 			)
 		)
-		(property "Manufacturer Part Number" ""
+		(property "Manufacturer Part Number" "VJ0603Y332KXBAC"
 			(at 106.68 58.42 0)
 			(effects
@@
 			)
 		)
-		(property "Footprint" "Capacitor_SMD:C_0603_1608Metric_Pad1.08x0.95mm_HandSolder"
+		(property "Footprint" "Resistor_SMD:R_0603_1608Metric_Pad0.98x0.95mm_HandSolder"
 			(at 96.52 51.562 90)
 			(effects
@@
 			)
 		)
-		(property "Description" ""
+		(property "Description" "ULM"
 			(at 96.52 53.34 0)
 			(effects
@@
 			)
 		)
-		(property "Manufacturer Part Number" ""
+		(property "Manufacturer Part Number" "CRCW060310K0FKEA"
 			(at 96.52 53.34 0)
 			(effects
@@
 			)
 		)
-		(property "Value" "1 uF"
+		(property "Value" "1uF"
 			(at 110.49 83.8199 0)
 			(effects
@@
 			)
 		)
-		(property "Description" ""
+		(property "Description" "ULM"
 			(at 106.68 82.55 0)
 			(effects
@@
 			)
 		)
-		(property "Manufacturer Part Number" ""
+		(property "Manufacturer Part Number" "C1206C105K5RACAUTO"
 			(at 106.68 82.55 0)
 			(effects

Commit message: BOM with Ullmanna part numbers
Parts:
- C2, C3: Manufacturer Part Number C1206C105K5RACAUTO -> CC603KRX5R8BB105; Mouser number 80-C1206C105K5RAUTO -> 603-CC603KRX5R8BB105; Ullmanna Part Number (none) -> BMCCK405
- R1, R2, R3: Manufacturer Part Number CRCW060310K0FKEA -> RC0603FR-0710KL; Mouser number 71-CRCW0603-10K-E3 -> 603-RC0603FR-0710KL; Ullmanna Part Number (none) -> BMCR0201
Changed lines of the file:
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@@
 (kicad_sch
-	(version 20231120)
+	(version 20250114)
 	(generator "eeschema")
-	(generator_version "8.0")
+	(generator_version "9.0")
 	(paper "A5")
 	(junction
@@
 		(shape bidirectional)
 		(at 106.68 40.64 270)
-		(fields_autoplaced yes)
 		(effects
 			(font
@@
 		(shape output)
 		(at 114.3 53.34 0)
-		(fields_autoplaced yes)
 		(effects
 			(font
@@
 		(shape input)
 		(at 87.63 53.34 180)
-		(fields_autoplaced yes)
 		(effects
 			(font
@@
 		(shape output)
 		(at 114.3 29.21 0)
-		(fields_autoplaced yes)
 		(effects
 			(font
@@
 		(shape output)
 		(at 114.3 77.47 0)
-		(fields_autoplaced yes)
 		(effects
 			(font
@@
 		(shape input)
 		(at 87.63 77.47 180)
-		(fields_autoplaced yes)
 		(effects
 			(font
@@
 		(shape bidirectional)
 		(at 106.68 64.77 270)
-		(fields_autoplaced yes)
 		(effects
 			(font
@@
 		(shape input)
 		(at 87.63 29.21 180)
-		(fields_autoplaced yes)
 		(effects
 			(font
@@
 		(shape bidirectional)
 		(at 106.68 88.9 270)
-		(fields_autoplaced yes)
 		(effects
 			(font
@@
 			)
 		)
-		(property "Manufacturer Part Number" "CRCW060310K0FKEA"
+		(property "Manufacturer Part Number" "RC0603FR-0710KL"
 			(at 96.52 29.21 0)
 			(effects
@@
 			)
 		)
-		(property "Mouser number" "71-CRCW0603-10K-E3"
+		(property "Mouser number" "603-RC0603FR-0710KL"
 			(at 96.52 29.21 0)
+			(effects
+				(font
+					(size 1.27 1.27)
+				)
+				(hide yes)
+			)
+		)
+		(property "Ullmanna Part Number" "BMCR0201"
+			(at 96.52 29.21 90)
 			(effects
 				(font
@@
 			)
 		)
-		(property "Manufacturer Part Number" "C1206C105K5RACAUTO"
+		(property "Manufacturer Part Number" "CC603KRX5R8BB105"
 			(at 106.68 34.29 0)
 			(effects
@@
 			)
 		)
-		(property "Mouser number" "80-C1206C105K5RAUTO"
+		(property "Mouser number" "603-CC603KRX5R8BB105"
+			(at 106.68 34.29 0)
+			(effects
+				(font
+					(size 1.27 1.27)
+				)
+				(hide yes)
+			)
+		)
+		(property "Ullmanna Part Number" "BMCCK405"
 			(at 106.68 34.29 0)
 			(effects
@@
 			)
 		)
-		(property "Manufacturer Part Number" "CRCW060310K0FKEA"
+		(property "Manufacturer Part Number" "RC0603FR-0710KL"
 			(at 96.52 77.47 0)
 			(effects
@@
 			)
 		)
-		(property "Mouser number" "71-CRCW0603-10K-E3"
+		(property "Mouser number" "603-RC0603FR-0710KL"
 			(at 96.52 77.47 0)
+			(effects
+				(font
+					(size 1.27 1.27)
+				)
+				(hide yes)
+			)
+		)
+		(property "Ullmanna Part Number" "BMCR0201"
+			(at 96.52 77.47 90)
 			(effects
 				(font
@@
 			)
 		)
+		(property "Ullmanna Part Number" ""
+			(at 106.68 58.42 0)
+			(effects
+				(font
+					(size 1.27 1.27)
+				)
+				(hide yes)
+			)
+		)
 		(pin "1"
 		)
@@
 			)
 		)
-		(property "Manufacturer Part Number" "CRCW060310K0FKEA"
+		(property "Manufacturer Part Number" "RC0603FR-0710KL"
 			(at 96.52 53.34 0)
 			(effects
@@
 			)
 		)
-		(property "Mouser number" "71-CRCW0603-10K-E3"
+		(property "Mouser number" "603-RC0603FR-0710KL"
 			(at 96.52 53.34 0)
+			(effects
+				(font
+					(size 1.27 1.27)
+				)
+				(hide yes)
+			)
+		)
+		(property "Ullmanna Part Number" "BMCR0201"
+			(at 96.52 53.34 90)
 			(effects
 				(font
@@
 			)
 		)
-		(property "Manufacturer Part Number" "C1206C105K5RACAUTO"
+		(property "Manufacturer Part Number" "CC603KRX5R8BB105"
 			(at 106.68 82.55 0)
 			(effects
@@
 			)
 		)
-		(property "Mouser number" "80-C1206C105K5RAUTO"
+		(property "Mouser number" "603-CC603KRX5R8BB105"
 			(at 106.68 82.55 0)
 			(effects
+				(font
+					(size 1.27 1.27)
+				)
+				(hide yes)
+			)
+		)
+		(property "Ullmanna Part Number" "BMCCK405"
+			(at 106.68 82.55 0)
+			(effects
