File: kicad/modules/MCU_module/MCU_module.kicad_pcb (KiCad board)
At the start: 2 copper layers, 33.3 x 64.1 mm, 17 parts, among them J1 Screw_Terminal_01x20, J2 Screw_Terminal_01x20, U1 Pico

Commit message: add control panel module
Other:
- board text added: "MCU_module"
- board text removed: "MCU_mudule"
Changed lines of the file:
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@@
 		)
 	)
-	(gr_text "MCU_mudule"
+	(gr_text "MCU_module"
 		(at 73.15 109.62 90)
 		(layer "F.SilkS")

Commit message: dots for orientation
Changed lines of the file:
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@@
 		(net 32)
+	)
+	(gr_circle
+		(center 102.3 114)
+		(end 103.3 114)
+		(stroke
+			(width 0.1)
+			(type solid)
+		)
+		(fill solid)
+		(layer "F.SilkS")
 	)
 	(gr_arc

Commit message: LED footprint update
Parts:
- C1: value 3.3 nF -> 3.3nF
- C2: value 1 uF -> 1uF
- C3: value none -> 1uF
- D1: footprint Diode_SMD:D_0603_1608Metric_Pad1.05x0.95mm_HandSolder -> Diode_SMD:D_0805_2012Metric_Pad1.15x1.40mm_HandSolder
- D2: renamed from POWER; footprint LED_SMD:LED_0603_1608Metric_Pad1.05x0.95mm_HandSolder -> LED_SMD:LED_0805_2012Metric_Pad1.15x1.40mm_HandSolder
- D3: renamed from STATUS; footprint LED_SMD:LED_0603_1608Metric_Pad1.05x0.95mm_HandSolder -> LED_SMD:LED_0805_2012Metric_Pad1.15x1.40mm_HandSolder
- ERROR: footprint LED_SMD:LED_0603_1608Metric_Pad1.05x0.95mm_HandSolder -> LED_SMD:LED_0805_2012Metric_Pad1.15x1.40mm_HandSolder
- J1, J2: value Screw_Terminal_01x20 -> 1x20, 2.54
- R1, R2: footprint Capacitor_SMD:C_0603_1608Metric_Pad1.08x0.95mm_HandSolder -> Resistor_SMD:R_0603_1608Metric_Pad0.98x0.95mm_HandSolder
- R3: value none -> 10k; footprint Capacitor_SMD:C_0603_1608Metric_Pad1.08x0.95mm_HandSolder -> Resistor_SMD:R_0603_1608Metric_Pad0.98x0.95mm_HandSolder
- SW1: renamed from RESET; value Reset -> BTN_RESET
- U1: value Pico -> RPI_PICO_2
Other:
- board text added: "POWER"
- board text added: "STATUS"
