File: kicad/modules/MCU_module/indicators.kicad_sch (KiCad schematic)
At the start: 6 parts

Commit message: Connector for bigger current, control module 2
Parts:
- D2: Mouser number (none) -> 78-VLMG1300-GS08
- D3: Mouser number (none) -> 78-VLMO1300-GS08
- D4: Mouser number (none) -> 78-VLMS1300-GS08
- R4, R5, R6: Mouser number (none) -> 71-CRCW0603-1.0K-E3
Changed lines of the file:
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@@
 			)
 		)
-		(property "Description" "78-VLMG1300-GS08"
+		(property "Description" ""
+			(at 85.09 67.31 0)
+			(effects
+				(font
+					(size 1.27 1.27)
+				)
+				(hide yes)
+			)
+		)
+		(property "Manufacturer Part Number" ""
+			(at 85.09 67.31 0)
+			(effects
+				(font
+					(size 1.27 1.27)
+				)
+				(hide yes)
+			)
+		)
+		(property "Mouser number" "78-VLMG1300-GS08"
 			(at 85.09 67.31 0)
 			(effects
@@
 			)
 		)
-		(property "Description" "78-VLMO1300-GS08"
+		(property "Description" ""
+			(at 101.6 67.31 0)
+			(effects
+				(font
+					(size 1.27 1.27)
+				)
+				(hide yes)
+			)
+		)
+		(property "Manufacturer Part Number" ""
+			(at 101.6 67.31 0)
+			(effects
+				(font
+					(size 1.27 1.27)
+				)
+				(hide yes)
+			)
+		)
+		(property "Mouser number" "78-VLMO1300-GS08"
 			(at 101.6 67.31 0)
 			(effects
@@
 			)
 		)
-		(property "Description" "71-CRCW0603-1.0K-E3"
+		(property "Description" ""
+			(at 101.6 59.69 0)
+			(effects
+				(font
+					(size 1.27 1.27)
+				)
+				(hide yes)
+			)
+		)
+		(property "Manufacturer Part Number" ""
+			(at 101.6 59.69 0)
+			(effects
+				(font
+					(size 1.27 1.27)
+				)
+				(hide yes)
+			)
+		)
+		(property "Mouser number" "71-CRCW0603-1.0K-E3"
 			(at 101.6 59.69 0)
 			(effects
@@
 			)
 		)
-		(property "Description" "71-CRCW0603-1.0K-E3"
+		(property "Description" ""
+			(at 118.11 59.69 0)
+			(effects
+				(font
+					(size 1.27 1.27)
+				)
+				(hide yes)
+			)
+		)
+		(property "Manufacturer Part Number" ""
+			(at 118.11 59.69 0)
+			(effects
+				(font
+					(size 1.27 1.27)
+				)
+				(hide yes)
+			)
+		)
+		(property "Mouser number" "71-CRCW0603-1.0K-E3"
 			(at 118.11 59.69 0)
 			(effects
@@
 			)
 		)
-		(property "Description" "78-VLMS1300-GS08"
+		(property "Description" ""
+			(at 118.11 67.31 0)
+			(effects
+				(font
+					(size 1.27 1.27)
+				)
+				(hide yes)
+			)
+		)
+		(property "Manufacturer Part Number" ""
+			(at 118.11 67.31 0)
+			(effects
+				(font
+					(size 1.27 1.27)
+				)
+				(hide yes)
+			)
+		)
+		(property "Mouser number" "78-VLMS1300-GS08"
 			(at 118.11 67.31 0)
 			(effects
@@
 			)
 		)
-		(property "Description" "71-CRCW0603-1.0K-E3"
+		(property "Description" ""
 			(at 85.09 59.69 0)
 			(effects
+				(font
+					(size 1.27 1.27)
+				)
+				(hide yes)
+			)
+		)
+		(property "Manufacturer Part Number" ""
+			(at 85.09 59.69 0)
+			(effects
+				(font
+					(size 1.27 1.27)
+				)
+				(hide yes)
+			)
+		)
+		(property "Mouser number" "71-CRCW0603-1.0K-E3"
+			(at 85.09 59.69 0)
+			(effects

Commit message: Add part numbers
Parts:
- D2: Manufacturer Part Number (none) -> VLMG1300-GS08
- D3: Manufacturer Part Number (none) -> VLMO1300-GS08
- D4: Manufacturer Part Number (none) -> VLMS1300-GS08
- R4, R5, R6: Manufacturer Part Number (none) -> CRCW06031K00FKEA
Changed lines of the file:
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@@
 			)
 		)
-		(property "Description" ""
+		(property "Description" "ULM"
 			(at 85.09 67.31 0)
 			(effects
@@
 			)
 		)
-		(property "Manufacturer Part Number" ""
+		(property "Manufacturer Part Number" "VLMG1300-GS08"
 			(at 85.09 67.31 0)
 			(effects
@@
 			)
 		)
-		(property "Description" ""
+		(property "Description" "ULM"
 			(at 101.6 67.31 0)
 			(effects
@@
 			)
 		)
-		(property "Manufacturer Part Number" ""
+		(property "Manufacturer Part Number" "VLMO1300-GS08"
 			(at 101.6 67.31 0)
 			(effects
@@
 			)
 		)
-		(property "Description" ""
+		(property "Description" "ULM"
 			(at 101.6 59.69 0)
 			(effects
@@
 			)
 		)
-		(property "Manufacturer Part Number" ""
+		(property "Manufacturer Part Number" "CRCW06031K00FKEA"
 			(at 101.6 59.69 0)
 			(effects
@@
 			)
 		)
-		(property "Description" ""
+		(property "Description" "ULM"
 			(at 118.11 59.69 0)
 			(effects
@@
 			)
 		)
-		(property "Manufacturer Part Number" ""
+		(property "Manufacturer Part Number" "CRCW06031K00FKEA"
 			(at 118.11 59.69 0)
 			(effects
@@
 			)
 		)
-		(property "Description" ""
+		(property "Description" "ULM"
 			(at 118.11 67.31 0)
 			(effects
@@
 			)
 		)
-		(property "Manufacturer Part Number" ""
+		(property "Manufacturer Part Number" "VLMS1300-GS08"
 			(at 118.11 67.31 0)
 			(effects
@@
 			)
 		)
-		(property "Description" ""
+		(property "Description" "ULM"
 			(at 85.09 59.69 0)
 			(effects
@@
 			)
 		)
-		(property "Manufacturer Part Number" ""
+		(property "Manufacturer Part Number" "CRCW06031K00FKEA"
 			(at 85.09 59.69 0)
 			(effects

Commit message: BOM with Ullmanna part numbers
Parts:
- D2: Manufacturer Part Number VLMG1300-GS08 -> APTD1608LCGCK; Mouser number 78-VLMG1300-GS08 -> 604-APTD1608LCGCK; Ullmanna Part Number (none) -> BMCLED002
- D3: Manufacturer Part Number VLMO1300-GS08 -> APTD1608LSYCK; Mouser number 78-VLMO1300-GS08 -> 604-APTD1608LSYCK; Ullmanna Part Number (none) -> BMCLED003
- D4: Manufacturer Part Number VLMS1300-GS08 -> APTD1608LSURCK; Mouser number 78-VLMS1300-GS08 -> 604-APTD1608LSURCK; Ullmanna Part Number (none) -> BMCLED004
- R4, R5, R6: Manufacturer Part Number CRCW06031K00FKEA -> RC0603FR-071KL; Mouser number 71-CRCW0603-1.0K-E3 -> 603-RC0603FR-071KL; Ullmanna Part Number (none) -> BMCR0176
Changed lines of the file:
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@@
 (kicad_sch
-	(version 20231120)
+	(version 20250114)
 	(generator "eeschema")
-	(generator_version "8.0")
+	(generator_version "9.0")
 	(paper "A5")
 	(wire
@@
 		(shape input)
 		(at 101.6 53.34 90)
-		(fields_autoplaced yes)
 		(effects
 			(font
@@
 		(shape input)
 		(at 85.09 53.34 90)
-		(fields_autoplaced yes)
 		(effects
 			(font
@@
 		(shape input)
 		(at 118.11 53.34 90)
-		(fields_autoplaced yes)
 		(effects
 			(font
@@
 			)
 		)
-		(property "Manufacturer Part Number" "VLMG1300-GS08"
+		(property "Manufacturer Part Number" "APTD1608LCGCK "
 			(at 85.09 67.31 0)
 			(effects
@@
 			)
 		)
-		(property "Mouser number" "78-VLMG1300-GS08"
+		(property "Mouser number" "604-APTD1608LCGCK"
+			(at 85.09 67.31 0)
+			(effects
+				(font
+					(size 1.27 1.27)
+				)
+				(hide yes)
+			)
+		)
+		(property "Ullmanna Part Number" "BMCLED002"
 			(at 85.09 67.31 0)
 			(effects
@@
 			)
 		)
-		(property "Manufacturer Part Number" "VLMO1300-GS08"
+		(property "Manufacturer Part Number" "APTD1608LSYCK"
 			(at 101.6 67.31 0)
 			(effects
@@
 			)
 		)
-		(property "Mouser number" "78-VLMO1300-GS08"
+		(property "Mouser number" "604-APTD1608LSYCK"
+			(at 101.6 67.31 0)
+			(effects
+				(font
+					(size 1.27 1.27)
+				)
+				(hide yes)
+			)
+		)
+		(property "Ullmanna Part Number" "BMCLED003"
 			(at 101.6 67.31 0)
 			(effects
@@
 			)
 		)
-		(property "Manufacturer Part Number" "CRCW06031K00FKEA"
+		(property "Manufacturer Part Number" "RC0603FR-071KL"
 			(at 101.6 59.69 0)
 			(effects
@@
 			)
 		)
-		(property "Mouser number" "71-CRCW0603-1.0K-E3"
+		(property "Mouser number" "603-RC0603FR-071KL"
+			(at 101.6 59.69 0)
+			(effects
+				(font
+					(size 1.27 1.27)
+				)
+				(hide yes)
+			)
+		)
+		(property "Ullmanna Part Number" "BMCR0176"
 			(at 101.6 59.69 0)
 			(effects
@@
 			)
 		)
-		(property "Manufacturer Part Number" "CRCW06031K00FKEA"
+		(property "Manufacturer Part Number" "RC0603FR-071KL"
 			(at 118.11 59.69 0)
 			(effects
@@
 			)
 		)
-		(property "Mouser number" "71-CRCW0603-1.0K-E3"
+		(property "Mouser number" "603-RC0603FR-071KL"
+			(at 118.11 59.69 0)
+			(effects
+				(font
+					(size 1.27 1.27)
+				)
+				(hide yes)
+			)
+		)
+		(property "Ullmanna Part Number" "BMCR0176"
 			(at 118.11 59.69 0)
 			(effects
@@
 			)
 		)
-		(property "Manufacturer Part Number" "VLMS1300-GS08"
+		(property "Manufacturer Part Number" "APTD1608LSURCK"
 			(at 118.11 67.31 0)
 			(effects
@@
 			)
 		)
-		(property "Mouser number" "78-VLMS1300-GS08"
+		(property "Mouser number" "604-APTD1608LSURCK"
+			(at 118.11 67.31 0)
+			(effects
+				(font
+					(size 1.27 1.27)
+				)
+				(hide yes)
+			)
+		)
+		(property "Ullmanna Part Number" "BMCLED004"
 			(at 118.11 67.31 0)
 			(effects
@@
 			)
 		)
-		(property "Manufacturer Part Number" "CRCW06031K00FKEA"
+		(property "Manufacturer Part Number" "RC0603FR-071KL"
 			(at 85.09 59.69 0)
 			(effects
@@
 			)
 		)
-		(property "Mouser number" "71-CRCW0603-1.0K-E3"
+		(property "Mouser number" "603-RC0603FR-071KL"
 			(at 85.09 59.69 0)
 			(effects
+				(font
+					(size 1.27 1.27)
+				)
+				(hide yes)
+			)
+		)
+		(property "Ullmanna Part Number" "BMCR0176"
+			(at 85.09 59.69 0)
+			(effects

Commit message: LED footprint update
Parts:
- D2: footprint LED_SMD:LED_0603_1608Metric_Pad1.05x0.95mm_HandSolder -> LED_SMD:LED_0805_2012Metric_Pad1.15x1.40mm_HandSolder; Manufacturer Part Number APTD1608LCGCK -> APTD2012LCGCK; Mouser number 604-APTD1608LCGCK -> 604-APTD2012LCGCK; Ullmanna Part Number BMCLED002 -> BMCLED102
- D3: footprint LED_SMD:LED_0603_1608Metric_Pad1.05x0.95mm_HandSolder -> LED_SMD:LED_0805_2012Metric_Pad1.15x1.40mm_HandSolder; Manufacturer Part Number APTD1608LSYCK -> APTD2012LSYCK; Mouser number 604-APTD1608LSYCK -> 604-APTD2012LSYCK; Ullmanna Part Number BMCLED003 -> BMCLED103
- D4: footprint LED_SMD:LED_0603_1608Metric_Pad1.05x0.95mm_HandSolder -> LED_SMD:LED_0805_2012Metric_Pad1.15x1.40mm_HandSolder; Manufacturer Part Number APTD1608LSURCK -> APTD2012LSURCK; Mouser number 604-APTD1608LSURCK -> 604-APTD2012LSURCK; Ullmanna Part Number BMCLED004 -> BMCLED104
Changed lines of the file:
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@@
 			)
 		)
-		(property "Footprint" "LED_SMD:LED_0603_1608Metric_Pad1.05x0.95mm_HandSolder"
+		(property "Footprint" "LED_SMD:LED_0805_2012Metric_Pad1.15x1.40mm_HandSolder"
 			(at 85.09 67.31 0)
 			(effects
@@
 			)
 		)
-		(property "Manufacturer Part Number" "APTD1608LCGCK "
+		(property "Manufacturer Part Number" "APTD2012LCGCK "
 			(at 85.09 67.31 0)
 			(effects
@@
 			)
 		)
-		(property "Mouser number" "604-APTD1608LCGCK"
+		(property "Mouser number" "604-APTD2012LCGCK "
 			(at 85.09 67.31 0)
 			(effects
@@
 			)
 		)
-		(property "Ullmanna Part Number" "BMCLED002"
+		(property "Ullmanna Part Number" "BMCLED102 "
 			(at 85.09 67.31 0)
 			(effects
@@
 			)
 		)
-		(property "Footprint" "LED_SMD:LED_0603_1608Metric_Pad1.05x0.95mm_HandSolder"
+		(property "Footprint" "LED_SMD:LED_0805_2012Metric_Pad1.15x1.40mm_HandSolder"
 			(at 101.6 67.31 0)
 			(effects
@@
 			)
 		)
-		(property "Manufacturer Part Number" "APTD1608LSYCK"
+		(property "Manufacturer Part Number" "APTD2012LSYCK "
 			(at 101.6 67.31 0)
 			(effects
@@
 			)
 		)
-		(property "Mouser number" "604-APTD1608LSYCK"
+		(property "Mouser number" "604-APTD2012LSYCK "
 			(at 101.6 67.31 0)
 			(effects
@@
 			)
 		)
-		(property "Ullmanna Part Number" "BMCLED003"
+		(property "Ullmanna Part Number" "BMCLED103 "
 			(at 101.6 67.31 0)
 			(effects
@@
 			)
 		)
-		(property "Footprint" "LED_SMD:LED_0603_1608Metric_Pad1.05x0.95mm_HandSolder"
+		(property "Footprint" "LED_SMD:LED_0805_2012Metric_Pad1.15x1.40mm_HandSolder"
 			(at 118.11 67.31 0)
 			(effects
@@
 			)
 		)
-		(property "Manufacturer Part Number" "APTD1608LSURCK"
+		(property "Manufacturer Part Number" "APTD2012LSURCK "
 			(at 118.11 67.31 0)
 			(effects
@@
 			)
 		)
-		(property "Mouser number" "604-APTD1608LSURCK"
+		(property "Mouser number" "604-APTD2012LSURCK "
 			(at 118.11 67.31 0)
 			(effects
@@
 			)
 		)
-		(property "Ullmanna Part Number" "BMCLED004"
+		(property "Ullmanna Part Number" "BMCLED104 "
 			(at 118.11 67.31 0)
 			(effects
