File: kicad/modules/DRV8874_module/DRV8874_module.kicad_pcb (KiCad board)
At the start: 2 copper layers, 45 x 23.5 mm, 48 parts, among them J1 SIGNALS, J2 POWER, U1 DRV8874PWPR

Commit message: LED footprint update
Parts:
- C4, C5: value 100 uF, 25V -> 100uF
- D1: value SS34A -> SS34
- D2: footprint LED_SMD:LED_0603_1608Metric_Pad1.05x0.95mm_HandSolder -> LED_SMD:LED_0805_2012Metric_Pad1.15x1.40mm_HandSolder
- F1: value 7.5 A -> FUSE 7.5 A
- J1: value SIGNALS -> 1x8 2.54
- J2: value POWER -> 1x8 2.54
- J3: renamed from OUT1; value MOTOR -> 1x2 5.08
Routing:
- added copper zone on F.Cu, net GND
