File: kicad/modules/DRV8874_module/power_supply.kicad_sch (KiCad schematic)
At the start: 4 parts

Commit message: LED footprint update
Parts:
- D2: footprint LED_SMD:LED_0603_1608Metric_Pad1.05x0.95mm_HandSolder -> LED_SMD:LED_0805_2012Metric_Pad1.15x1.40mm_HandSolder; Manufacturer Part Number APTD1608LCGCK -> APTD2012LCGCK; Mouser number 604-APTD1608LCGCK -> 604-APTD2012LCGCK; Ullmanna Part Number BMCLED002 -> BMCLED102
Changed lines of the file:
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@@
 			)
 		)
-		(property "Footprint" "LED_SMD:LED_0603_1608Metric_Pad1.05x0.95mm_HandSolder"
+		(property "Footprint" "LED_SMD:LED_0805_2012Metric_Pad1.15x1.40mm_HandSolder"
 			(at 48.26 40.64 0)
 			(effects
@@
 			)
 		)
-		(property "Manufacturer Part Number" "APTD1608LCGCK "
+		(property "Manufacturer Part Number" "APTD2012LCGCK "
 			(at 48.26 40.64 0)
 			(effects
@@
 			)
 		)
-		(property "Mouser number" "604-APTD1608LCGCK "
+		(property "Mouser number" "604-APTD2012LCGCK "
 			(at 48.26 40.64 0)
 			(effects
@@
 			)
 		)
-		(property "Ullmanna Part Number" "BMCLED002 "
+		(property "Ullmanna Part Number" "BMCLED102 "
 			(at 48.26 40.64 90)
 			(effects
